File: space-invader.kicad_pcb (KiCad board)
At the start: 2 copper layers, 95.3 x 81 mm, 39 parts, among them SW1 SW_Push, SW10 SW_Push, SW11 SW_Push, SW12 SW_Push, SW13 SW_Push, SW14 SW_Push, SW15 SW_Push, SW16 SW_Push, SW17 SW_Push, SW2 SW_Push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

Commit message: added on-off switch
Parts:
- added BAT+: BAT+_Pad, TestPoint:TestPoint_Pad_1.5x1.5mm, F.Cu at (74.9, 94.0)
- added MCU+: BAT+_Pad_MCU, TestPoint:TestPoint_Pad_1.5x1.5mm, F.Cu at (77.5, 94.0)
- added SW18: SW_SPDT, PCM_marbastlib-various:SW_MSK12C02-HB, B.Cu at (76.2, 98.0)
- moved kibuzzard-67AF24D7 1.40 mm to (65.3, 97.7)
Connections:
- U1 pad 15: BAT- -> unconnected-(U1-BAT--Pad15)
- U1 pad 16: BAT+ -> unconnected-(U1-BAT+-Pad16)
Routing:
- net BAT+MCU: track 0.00 -> 5.87 mm, vias 0 -> 1
- net BAT+: track 0.00 -> 4.96 mm, vias 0 -> 1
- added copper zone on B.Cu, net BAT+MCU
- added copper zone on F.Cu, net BAT+MCU
- removed copper zone on B.Cu, net (none)
- removed copper zone on F.Cu, net (none)
